File: HydraBus_1_0_Rev1_1.brd (EAGLE design)
At the start: 60 x 37 mm, 60 parts, among them IC1 STM32F405RGT, J1 CON_HEADER_2X06, J2 CON_HEADER_2X08, J3 CON_HEADER_2X08, J4 MICRO-SDCARD-CONNECTOR-330006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, J5 CON_HEADER_1X06-PTH, U1 IP4220CZ6, Y1_8MHZ 631-1100-ND, Y2_32.768KHZ 32.768KHz

Commit message: Updated .sch and .brd
Parts:
- R7: value 2.2K -> 10K
- moved R7 15.8 mm to (47.8, 15.0), turned to 90 degrees
Connections:
- removed net N$9: JMP1.4, R12.2
- net BOOT0: now also JMP1.4, R12.2; no longer R7.1
- net PB2: now also R7.1
Routing:
- net BOOT0: track 26.3 -> 48.1 mm, vias 3 -> 6
- net N$9: track 7.76 -> 0.00 mm
- net GND: track 39.4 -> 43.2 mm, vias 65 -> 91
- net N$6: track 14.4 -> 12.1 mm
- net +3V3: track 228.1 -> 229.8 mm
- net NRST: track 61.4 -> 60.5 mm
Other:
- board text added: "(C) B.VERNOUX v1.0 Rev1_2"
- board text added: "/BOOT DFU"
- board text added: "NC"
- board text removed: "(C) B.VERNOUX v1.0 Rev1_1"
- board text removed: "ADC1_IN0"
- board text removed: "ADC2_IN1"
- board text removed: "ADC3_IN10"
- board text removed: "BOOT1"
- board text removed: "DAC1_OUT"
- board text removed: "DAC2_OUT"
- board text removed: "I2C1_SCL"
- board text removed: "I2C1_SDA"
- board text removed: "SDIO_CK"
- board text removed: "SDIO_CMD"
- board text removed: "SDIO_D0"
- board text removed: "SDIO_D1"
- board text removed: "SDIO_D2"
- board text removed: "SDIO_D3"
- board text removed: "SPI1_MISO"
- board text removed: "SPI1_MOSI"
- board text removed: "SPI1_NSS"
- board text removed: "SPI1_SCK"
- board text removed: "SPI2_MISO"
- board text removed: "SPI2_SCK"
- board text removed: "USART1_CK"
- board text removed: "USART1_RX"
- board text removed: "USART1_TX"
- board text removed: "USART2_RX"
- board text removed: "USART2_TX"
- board text removed: "USB0_D+"
- board text removed: "USB0_D-"
